Commit message: update xacro property

File: ROS2_basic/my_robot_description/urdf/my_robot.urdf.xacro (robot description, xacro)
@@ -1,5 +1,10 @@
 <?xml version="1.0"?>
 <robot name="my_robot" xmlns:xacro="http://www.ros.org/wiki/xacro">
-    <xacro:property name="base_length" value="1.0" />
+    <xacro:property name="base_length" value="0.6" />
+    <xacro:property name="base_width" value="0.4" />
+    <xacro:property name="base_radius" value="1.0" />
+    <xacro:property name="base_height" value="0.2" />
+    <xacro:property name="wheel_radius" value="0.1" />
+    <xacro:property name="wheel_length" value="0.05" />
     <material name="grey">
         <color rgba="0.7 0.7 0.7 1.0"/>
@@ -19,7 +24,7 @@
         <visual>
             <geometry>
-                <box size="${base_length} 0.4 0.2"/>
+                <box size="${base_length} ${base_width} ${base_height}"/>
             </geometry>
-            <origin xyz="0.0 0.0 0.1" rpy="0.0 0.0 0.0"/>
+            <origin xyz="0.0 0.0 ${base_height / 2.0}" rpy="0.0 0.0 0.0"/>
             <material name="green"/>
         </visual>
@@ -38,5 +43,5 @@
             <origin xyz="0.0 0.0 0.0" rpy="${pi / 2} 0.0 0.0"/>
             <geometry>
-                <cylinder radius="0.1" length="0.05"/>
+                <cylinder radius="${wheel_radius}" length="${wheel_length}"/>
             </geometry>
             <material name="grey"/>
@@ -47,14 +52,14 @@
             <origin xyz="0.0 0.0 0.0" rpy="${pi / 2.0} 0.0 0.0"/>
             <geometry>
-                <cylinder radius="0.1" length="0.05"/>
+                <cylinder radius="${wheel_radius}" length="${wheel_length}"/>
             </geometry>
             <material name="grey"/>
         </visual>
     </link>
-    <link name="caster_wheel">
+    <link name="caster_wheel_link">
         <visual>
             <origin xyz="0.0 0.0 0.0" rpy="0.0 0.0 0.0"/>
             <geometry>
-                <sphere radius="0.05"/>
+                <sphere radius="${wheel_radius / 2.0}"/>
             </geometry>
             <material name="grey"/>
@@ -67,5 +72,5 @@
     </joint>
     <joint name="base_left_wheel_joint" type="continuous">
-        <origin xyz="${-base_length / 4.0} 0.225 0.0" rpy="0.0 0.0 0.0"/>
+        <origin xyz="${-base_length / 4.0} ${(base_width + wheel_length) / 2.0} 0.0" rpy="0.0 0.0 0.0"/>
         <parent link="base_link"/>
         <child link="left_wheel"/>
@@ -73,5 +78,5 @@
     </joint>
     <joint name="base_right_wheel_joint" type="continuous">
-        <origin xyz="${-base_length / 4.0} -0.225 0.0" rpy="0.0 0.0 0.0"/>
+        <origin xyz="${-base_length / 4.0} ${-(base_width + wheel_length) / 2.0} 0.0" rpy="0.0 0.0 0.0"/>
         <parent link="base_link"/>
         <child link="right_wheel"/>
@@ -79,12 +84,12 @@
     </joint>
     <joint name="base_caster_wheel_joint" type="fixed">
-        <origin xyz="${base_length / 3.0} 0.0 -0.05" rpy="0.0 0.0 0.0"/>
+        <origin xyz="${base_length / 3.0} 0.0 -${wheel_radius / 2.0}" rpy="0.0 0.0 0.0"/>
         <parent link="base_link"/>
-        <child link="caster_wheel"/>
+        <child link="caster_wheel_link"/>
     </joint>
     <joint name="base_joint" type="fixed">
         <parent link="base_footprint"/>
         <child link="base_link"/>
-        <origin xyz="0.0 0.0 0.1" rpy="0.0 0.0 0.0"/>
+        <origin xyz="0.0 0.0 ${wheel_radius}" rpy="0.0 0.0 0.0"/>
     </joint>
 </robot>
