Commit message: update xacro

File: ROS2_basic/my_robot_description/urdf/my_robot2_include.urdf.xacro (robot description, xacro)
@@ -1,4 +1,5 @@
 <?xml version="1.0"?>
 <robot name="my_robot" xmlns:xacro="http://www.ros.org/wiki/xacro">
+    <xacro:include filename="common_properties.xacro"/>
     <xacro:property name="base_length" value="0.6" />
     <xacro:property name="base_width" value="0.4" />
@@ -7,26 +8,4 @@
     <xacro:property name="wheel_radius" value="0.1" />
     <xacro:property name="wheel_length" value="0.05" />
-    <!-- <xacro:macro name="example_macro" params="a b c">
-        <link name="dummy_link">
-            <visual>
-                <geometry>
-                    <box size="${a} ${b} ${c}"/>
-                </geometry>
-            </visual>
-        </link>
-    </xacro:macro>
-    <xacro:example_macro a="2" b="3" c="4" /> -->
-    <material name="grey">
-        <color rgba="0.7 0.7 0.7 1.0"/>
-    </material>
-    <material name="blue">
-        <color rgba="0.0 0.5 1.0 1.0"/>
-    </material>
-    <material name="green">
-        <color rgba="0.0 0.6 0.0 1.0"/>
-    </material>
-    <material name="white">
-        <color rgba="1.0 1.0 1.0 1.0"/>
-    </material>
     <link name="base_footprint">
     </link>
@@ -49,18 +28,5 @@
         </visual>
     </link>
-    <xacro:macro name="wheel_link" params="prefix">
-        <link name="${prefix}_wheel_link" >
-            <visual>
-            <origin xyz="0.0 0.0 0.0" rpy="${pi / 2} 0.0 0.0"/>
-            <geometry>
-                <cylinder radius="${wheel_radius}" length="${wheel_length}"/>
-            </geometry>
-            <material name="grey"/>
-            </visual>
-        </link>
-    </xacro:macro>
-    <xacro:wheeel_link prefix="right" />
-    <xacro:wheeel_link prefix="left" />
-    <!-- <link name="left_wheel_link">
+    <link name="left_wheel">
         <visual>
             <origin xyz="0.0 0.0 0.0" rpy="${pi / 2} 0.0 0.0"/>
@@ -71,5 +37,5 @@
         </visual>
     </link>
-    <link name="right_wheel_link">
+    <link name="right_wheel">
         <visual>
             <origin xyz="0.0 0.0 0.0" rpy="${pi / 2.0} 0.0 0.0"/>
@@ -79,5 +45,5 @@
             <material name="grey"/>
         </visual>
-    </link> -->
+    </link>
     <link name="caster_wheel_link">
         <visual>
@@ -97,5 +63,5 @@
         <origin xyz="${-base_length / 4.0} ${(base_width + wheel_length) / 2.0} 0.0" rpy="0.0 0.0 0.0"/>
         <parent link="base_link"/>
-        <child link="left_wheel_link"/>
+        <child link="left_wheel"/>
         <axis xyz="0.0 1.0 0.0"/>
     </joint>
@@ -103,5 +69,5 @@
         <origin xyz="${-base_length / 4.0} ${-(base_width + wheel_length) / 2.0} 0.0" rpy="0.0 0.0 0.0"/>
         <parent link="base_link"/>
-        <child link="right_wheel_link"/>
+        <child link="right_wheel"/>
         <axis xyz="0.0 1.0 0.0"/>
     </joint>
