Commit message: xacro include debug

File: ROS2_basic/my_robot_description/urdf/my_robot2.urdf.xacro (robot description, xacro)
@@ -1,4 +1,4 @@
 <?xml version="1.0"?>
-<robot xmlns:xacro="http://www.ros.org/wiki/xacro">
+<robot name="my_robot2" xmlns:xacro="http://www.ros.org/wiki/xacro">
     <xacro:property name="base_length" value="0.6" />
     <xacro:property name="base_width" value="0.4" />
@@ -7,5 +7,6 @@
     <xacro:property name="wheel_radius" value="0.1" />
     <xacro:property name="wheel_length" value="0.05" />
-    <material name="grey">
+    <xacro:include filename="common_properties.xacro"/>
+    <!-- <material name="grey">
         <color rgba="0.7 0.7 0.7 1.0"/>
     </material>
@@ -18,5 +19,5 @@
     <material name="white">
         <color rgba="1.0 1.0 1.0 1.0"/>
-    </material>
+    </material> -->
     <link name="base_footprint">
     </link>
