Commit message: add 6-1 solution

File: ROS2_basic/my_robot_description/urdf/common_properties.xacro (robot description, xacro)
@@ -13,3 +13,29 @@
         <color rgba="1.0 1.0 1.0 1.0"/>
     </material>
+    <xacro:macro name="box_inertia" params="m l w h xyz rpy">
+        <inertial>
+            <origin xyz="${xyz}" rpy="${rpy}"/>
+            <mass value="${m}" />
+            <inertial ixx="${(m/12) * (h*h + l*l)}" ixy="0" ixz="0"
+                      iyy="${(m/12) * (w*w + l*l)}" iyz="0"
+                      izz="${(m/12) * (w*w + h*h)}" />
+        </inertial>
+    </xacro:macro>
+    <xacro:macro name="cylinder_inertia" params="m r h xyz rpy">
+        <inertial>
+        <origin xyz="${xyz}" rpy="${rpy}" />
+        <mass value="${m}" />
+        <inertial ixx="${(m/12) * (3*r*r + h*h)}" ixy="0" ixz="0"
+                  iyy="${(m/12) * (3*r*r + h*h)}" iyz="0"
+                  izz="${(m/2) * (r*r)}" />
+    </xacro:macro>
+    <xacro:macro name="sphere_inertia" params="m r xyz rpy">
+        <inertial>
+            <origin xyz="${xyz}" rpy="${rpy}"/>
+            <mass value="${m}" />
+            <inertial ixx="${(2/5 * m * r * r)}" ixy="0" ixz="0"
+                      iyy="${(2/5 * m * r * r)}" iyz="0"
+                      izz="${(2/5 * m * r * r)}" />
+        </inertial>
+    </xacro:macro>
 </robot>

File: ROS2_basic/my_robot_description/urdf/robot_inertia.urdf.xacro (robot description, xacro)
@@ -8,16 +8,4 @@
     <xacro:property name="wheel_length" value="0.05" />
     <xacro:include filename="common_properties.xacro"/>
-    <!-- <material name="grey">
-        <color rgba="0.7 0.7 0.7 1.0"/>
-    </material>
-    <material name="blue">
-        <color rgba="0.0 0.5 1.0 1.0"/>
-    </material>
-    <material name="green">
-        <color rgba="0.0 0.6 0.0 1.0"/>
-    </material>
-    <material name="white">
-        <color rgba="1.0 1.0 1.0 1.0"/>
-    </material> -->
     <link name="base_footprint">
     </link>
@@ -30,4 +18,12 @@
             <material name="green"/>
         </visual>
+        <collision>
+           <geometry>
+                <box size="${base_length} ${base_width} ${base_height}"/>
+            </geometry>
+            <origin xyz="0.0 0.0 ${base_height / 2.0}" rpy="0.0 0.0 0.0"/>
+        </collision>
+        <xacro:box_inertia m="5.0" l="${base_length}" w="${base_width}" h="${base_height}"
+                           xyz="0 0 ${base_height / 2.0}" rpy="{0 0 0}" />
     </link>
     <link name="lidar">
@@ -48,4 +44,6 @@
             <material name="grey"/>
         </visual>
+        <xacro:cylinder_inertia m="1.0" r="${wheel_radius}" h="${wheel_length}"
+                                xyz="0 0 0" rpy="${pi / 2.0} 0 0" />
     </link>
     <link name="right_wheel">
@@ -66,4 +64,6 @@
             <material name="grey"/>
         </visual>
+        <xacro:sphere_inertia m="0.5" r="${wheel_radius / 2.0}"
+                              xyz="0 0 0" rpy="0 0 0" />
     </link>
     <joint name="base_lidar_joint" type="fixed">
